Commit message: WIP joint control

File: src/cmg_leg_description/urdf/robot_body_roll.urdf (robot description, URDF)
Before this commit: robot wheeled_inverted_pendulum, 11 links, 10 joints
Links:
- link Left_flywheel: geometry collision mesh filename=package://cmg_leg_description/meshes/left_flywheel_link.STL scale=0.001 0.001 0.001; visual mesh filename=package://cmg_leg_description/meshes/left_flywheel_link.STL scale=0.001 0.001 0.001
- link Left_gimbal: geometry collision mesh filename=package://cmg_leg_description/meshes/left_gimbal_link.STL scale=0.001 0.001 0.001; visual mesh filename=package://cmg_leg_description/meshes/left_gimbal_link.STL scale=0.001 0.001 0.001
- link Right_flywheel: geometry collision mesh filename=package://cmg_leg_description/meshes/right_flywheel_link.STL scale=0.001 0.001 0.001; visual mesh filename=package://cmg_leg_description/meshes/right_flywheel_link.STL scale=0.001 0.001 0.001
- link Right_gimbal: geometry collision mesh filename=package://cmg_leg_description/meshes/right_gimbal_link.STL scale=0.001 0.001 0.001; visual mesh filename=package://cmg_leg_description/meshes/right_gimbal_link.STL scale=0.001 0.001 0.001
- link ankle_link: geometry collision mesh filename=package://cmg_leg_description/meshes/ankle_link.STL scale=0.001 0.001 0.001; visual mesh filename=package://cmg_leg_description/meshes/ankle_link.STL scale=0.001 0.001 0.001
- link frame: geometry collision mesh filename=package://cmg_leg_description/meshes/cmg_link.STL scale=0.001 0.001 0.001; visual mesh filename=package://cmg_leg_description/meshes/cmg_link.STL scale=0.001 0.001 0.001
- link hip_link: geometry collision mesh filename=package://cmg_leg_description/meshes/hip_link.STL scale=0.001 0.001 0.001; visual mesh filename=package://cmg_leg_description/meshes/hip_link.STL scale=0.001 0.001 0.001
- link hip_to_knee_link: geometry collision mesh filename=package://cmg_leg_description/meshes/hip_to_knee_link.STL scale=0.001 0.001 0.001; visual mesh filename=package://cmg_leg_description/meshes/hip_to_knee_link.STL scale=0.001 0.001 0.001
- link knee_ankle_link: geometry collision mesh filename=package://cmg_leg_description/meshes/knee_to_ankle_pitch_li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 scale=0.001 0.001 0.001; visual mesh filename=package://cmg_leg_description/meshes/knee_to_ankle_pitch_li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 scale=0.001 0.001 0.001
- link wheel_link: geometry collision mesh filename=package://cmg_leg_description/meshes/wheel_link.STL scale=0.001 0.001 0.001; visual mesh filename=package://cmg_leg_description/meshes/wheel_link.STL scale=0.001 0.001 0.001
Joints:
- joint ankle_pitch_joint: limit lower=0 upper=0 effort=100 velocity=1000 -> lower=0.1 upper=2.5 effort=1000 velocity=1000; origin xyz=0 0 -0.279942 rpy=0.0 0.0 0.0 -> xyz=0 0 -0.279942 rpy=0.0 -0.7577 0.0
- joint hip_pitch_joint: limit lower=0 upper=0 effort=100 velocity=1000 -> lower=0.1 upper=2.5 effort=1000 velocity=1000; origin xyz=0 0 0 rpy=0.0 0 0.0 -> xyz=0 0 0 rpy=0.0 -0.8744 0.0
- joint knee_joint: limit lower=0 upper=0 effort=100 velocity=1000 -> lower=-3.0 upper=-0.1 effort=1000 velocity=1000; origin xyz=0 0 -0.28 rpy=0.0 0 0.0 -> xyz=0 0 -0.28 rpy=0.0 1.6321 0.0
