Commit message: WIP joint control

File: src/cmg_leg_description/urdf/robot.urdf (robot description, URDF)
Before this commit: robot wheeled_inverted_pendulum, 11 links, 10 joints
Joints:
- joint ankle_pitch_joint: origin xyz=0 0 -0.279942 rpy=0.0 -0.755239 0.0 -> xyz=0 0 -0.279942 rpy=0.0 0 0.0
- joint cmg_joint: origin xyz=0 0 0.8452 rpy=0.0 0.0 0.0 -> xyz=0 0 1.022142 rpy=0.0 0.0 0.0
- joint hip_pitch_joint: origin xyz=0 0 0 rpy=0.0 -0.885463 0.0 -> xyz=0 0 0 rpy=0.0 0 0.0
- joint knee_joint: origin xyz=0 0 -0.28 rpy=0.0 1.6307 0.0 -> xyz=0 0 -0.28 rpy=0.0 0 0.0

Commit message: CUIP joint control

File: src/cmg_leg_description/urdf/robot.urdf (robot description, URDF)
Before this commit: robot wheeled_inverted_pendulum, 11 links, 10 joints
Links:
- removed link frame
- removed link hip_link
- added link cmg_hip_link, mass 7.774; collision mesh filename=package://cmg_leg_description/meshes/cmg_hip_link.STL scale=0.001 0.001 0.001; visual mesh filename=package://cmg_leg_description/meshes/cmg_hip_link.STL scale=0.001 0.001 0.001
- link Left_flywheel: mass 4 -> 3.73
- link Left_gimbal: mass 1 -> 0.92
- link Right_flywheel: mass 4 -> 3.73
- link Right_gimbal: mass 1 -> 0.92
- link ankle_link: mass 2.786 -> 2.486
Joints:
- removed joint cmg_joint
- removed joint hip_roll_joint
- added joint cmg_hip_joint: type fixed, parent cmg, child cmg_hip_link, origin xyz=0 0 1.022142 rpy=0.0 0.0 0.0
- joint Left_gimbal_joint: parent frame -> cmg_hip_link
- joint Right_gimbal_joint: parent frame -> cmg_hip_link
- joint hip_pitch_joint: origin xyz=0 0 0 rpy=0.0 0 0.0 -> xyz=0 0 -0.2222 rpy=0.0 0 0.0; parent hip_link -> cmg_hip_link

Commit message: WIP joint control

File: src/cmg_leg_description/urdf/robot.urdf (robot description, URDF)
Before this commit: robot wheeled_inverted_pendulum, 10 links, 9 joints
Joints:
- joint ankle_pitch_joint: limit lower=-1.5 upper=0.0 effort=1000 velocity=1000 -> effort=1000 velocity=1000; origin xyz=0 0 -0.279942 rpy=0.0 0 0.0 -> xyz=0 0 -0.279942 rpy=0.0 -0.745238866846359 0.0; type revolute -> continuous
- joint cmg_hip_joint: origin xyz=0 0 1.022142 rpy=0.0 0.0 0.0 -> xyz=0 0 0.845 rpy=0.0 0.0 0.0
- joint hip_pitch_joint: limit lower=-1.57 upper=0 effort=1000 velocity=1000 -> effort=1000 velocity=1000; origin xyz=0 0 -0.2222 rpy=0.0 0 0.0 -> xyz=0 0 -0.2222 rpy=0.0 -0.885462876712376 0.0; type revolute -> continuous
- joint knee_joint: limit lower=0.0 upper=2.4 effort=1000 velocity=1000 -> effort=1000 velocity=1000; origin xyz=0 0 -0.28 rpy=0.0 0 0.0 -> xyz=0 0 -0.28 rpy=0.0 1.63070174355873 0.0; type revolute -> continuous
