Commit message: WIP joint control

File: src/cmg_leg_description/urdf/cmg_joint.urdf (robot description, URDF)
Before this commit: robot wheeled_inverted_pendulum, 11 links, 10 joints
Joints:
- joint ankle_pitch_joint: limit lower=0.1 upper=2.5 effort=1000 velocity=1000 -> lower=0 upper=0 effort=1000 velocity=1000
- joint cmg_joint: axis 0 1 0 -> (none); limit effort=100 velocity=1000 -> (none); type continuous -> fixed
- joint hip_pitch_joint: limit lower=0.1 upper=2.5 effort=1000 velocity=1000 -> lower=0.0 upper=0 effort=1000 velocity=1000
- joint knee_joint: limit lower=-3.0 upper=-0.1 effort=1000 velocity=1000 -> lower=0 upper=0 effort=1000 velocity=1000
- joint wheel_joint: limit lower=0.1 upper=2.5 effort=100 velocity=1000 -> lower=0.0 upper=0 effort=100 velocity=1000; origin xyz=0 0 0.0 rpy=0.0 0.0 0.0 -> xyz=0 0 0.171 rpy=0.0 0.0 0.0

File: src/cmg_leg_description/urdf/robot.urdf (robot description, URDF)
Before this commit: robot wheeled_inverted_pendulum, 11 links, 10 joints
Joints:
- joint ankle_pitch_joint: limit lower=0.1 upper=2.5 effort=1000 velocity=1000 -> lower=-1.5 upper=0.0 effort=1000 velocity=1000; origin xyz=0 0 -0.279942 rpy=0.0 -0.7577 0.0 -> xyz=0 0 -0.279942 rpy=0.0 -0.755239 0.0
- joint cmg_joint: origin xyz=0 0 1.022142 rpy=0.0 0.0 0.0 -> xyz=0 0 0.8452 rpy=0.0 0.0 0.0
- joint hip_pitch_joint: limit lower=0.1 upper=2.5 effort=1000 velocity=1000 -> lower=-1.57 upper=0 effort=1000 velocity=1000; origin xyz=0 0 0 rpy=0.0 -0.8744 0.0 -> xyz=0 0 0 rpy=0.0 -0.885463 0.0
- joint knee_joint: limit lower=-3.0 upper=-0.1 effort=1000 velocity=1000 -> lower=0.0 upper=2.4 effort=1000 velocity=1000; origin xyz=0 0 -0.28 rpy=0.0 1.6321 0.0 -> xyz=0 0 -0.28 rpy=0.0 1.6307 0.0
- joint wheel_joint: limit effort=100 velocity=1000 -> effort=1000 velocity=1000

Commit message: WIP joint

File: src/cmg_leg_description/urdf/cmg_joint.urdf (robot description, URDF)
Before this commit: robot wheeled_inverted_pendulum, 11 links, 10 joints
Links:
- removed link frame
- removed link hip_link
- removed link wheel
- added link ankle
- added link cmg_hip_link, mass 7.774; collision mesh filename=package://cmg_leg_description/meshes/cmg_hip_link.STL scale=0.001 0.001 0.001; visual mesh filename=package://cmg_leg_description/meshes/cmg_hip_link.STL scale=0.001 0.001 0.001
- added link imu_link
- link Left_flywheel: mass 4 -> 3.73
- link Left_gimbal: mass 1 -> 0.92
- link Right_flywheel: mass 4 -> 3.73
- link Right_gimbal: mass 1 -> 0.92
Joints:
- removed joint hip_roll_joint
- added joint imu_joint: type revolute, parent cmg_hip_link, child imu_link, origin xyz=0 0 0.28 rpy=0.0 0.0 0.0, axis 0 0 1, limit lower=0.0 upper=0 effort=1000 velocity=1000
- joint Left_gimbal_joint: origin xyz=0 0.08 0 rpy=0 0 0 -> xyz=0 0.08 0.222 rpy=0 0 0; parent frame -> cmg_hip_link
- joint Right_gimbal_joint: origin xyz=0 -0.08 0 rpy=0 0 0 -> xyz=0 -0.08 0.222 rpy=0 0 0; parent frame -> cmg_hip_link
- joint ankle_pitch_joint: limit lower=0 upper=0 effort=1000 velocity=1000 -> lower=-1 upper=1 effort=1000 velocity=1000; origin xyz=0 0 0.279942 rpy=0.0 0 0.0 -> xyz=0 0 0.0 rpy=0.0 0.745238866846359 0.0
- joint cmg_joint: child wheel_link -> ankle_link; origin xyz=0 0 0.069 rpy=0.0 0.0 0.0 -> xyz=0 0 0.24 rpy=0.0 0.0 0.0; parent wheel -> ankle
- joint hip_pitch_joint: axis 0 1 0 -> (none); child hip_link -> cmg_hip_link; limit lower=0.0 upper=0 effort=1000 velocity=1000 -> (none); origin xyz=0 0 0 rpy=0.0 0 0.0 -> xyz=0 0 0.28 rpy=0.0 0.885462876712376 0.0; type revolute -> fixed
- joint knee_joint: axis 0 1 0 -> (none); limit lower=0 upper=0 effort=1000 velocity=1000 -> (none); origin xyz=0 0 0.28 rpy=0.0 0 0.0 -> xyz=0 0 0.279942 rpy=0.0 -1.63070174355873 0.0; type revolute -> fixed
- joint wheel_joint: child ankle_link -> wheel_link; origin xyz=0 0 0.171 rpy=0.0 0.0 0.0 -> xyz=0 0 -0.171 rpy=0.0 0.0 0.0; parent wheel_link -> ankle_link; type revolute -> continuous

File: src/cmg_leg_description/urdf/robot.urdf (robot description, URDF)
Before this commit: robot wheeled_inverted_pendulum, 10 links, 9 joints
Joints:
- joint ankle_pitch_joint: limit effort=1000 velocity=1000 -> lower=-1 upper=1 effort=1000 velocity=1000; type continuous -> revolute
- joint hip_pitch_joint: limit effort=1000 velocity=1000 -> (none); type continuous -> fixed
- joint knee_joint: limit effort=1000 velocity=1000 -> (none); type continuous -> fixed
